File: hardware/ir-rf-blaster-hat/xiao-c3-ir-rf.kicad_pcb (KiCad board)
At the start: 4 copper layers, 23 x 54 mm, 15 parts, among them M1 E07-M1101D, Q1 AO3400A

Commit message: fix(ir-blaster): move IR_TX off GPIO2 strapping pin to D1/GPIO3
Pre-fab review caught that IR_TX sat on D0/GPIO2 — an ESP32-C3 strapping pin —
and the 10k gate pulldown drags GPIO2 to ~0.6V at reset (through the ~45k
internal pull-up), against Espressif's strapping guidance (boot reliability
risk). D1/GPIO3 is spare and non-strapping, so move IR_TX there; all three
strapping pins (D0/D8/D9) are now left spare. Zero cost, still DRC 0/0.

Regenerated board + gerbers + renders; README pin map + firmware pin (GPIO3)
updated.

Co-Authored-By: Claude Opus 4.8 <noreply@anthropic.com>
Claude-Session: https://claude.ai/code/session_01NfkRErMrPyNuft1RbpzMet
Connections:
- A1 pad 1: IR_TX -> (no net)
- A1 pad 2: (no net) -> IR_TX
Routing:
- net IR_TX: track 27.2 -> 34.4 mm
